File: sensors/reed-level-sensing/reed-level-sensing.kicad_sch (KiCad schematic)
At the start: 0 parts

Commit message: Worked on KiKad schematic 10/28/26
Parts:
- added C1, C2: 100n, Package_SO:SOIC-8_3.9x4.9mm_P1.27mm, symbol Device:C
- added C3: 10u, Package_SO:SOIC-8_3.9x4.9mm_P1.27mm, symbol Device:C
- added D1: LED, Package_TO_SOT_SMD:SOT-323_SC-70, symbol Device:LED
- added J1: Conn_01x04_Pin, symbol Connector:Conn_01x04_Pin
- added R1: 1k, symbol Device:R
- added R2: 56, symbol Device:R
- added U1: ADS1013IDGS, Package_SO:TSSOP-10_3x3mm_P0.5mm, symbol Analog_ADC:ADS1013IDGS
- added U2: TPD2E2U06DCK, Package_TO_SOT_SMD:SOT-323_SC-70, symbol Power_Protection:TPD2E2U06DCK
Connections:
- new net: C1.1, C3.1, J1.1 (Pin_1), R2.2, U1.8 (VDD)
- new net: C1.2, C2.2, C3.2, J1.4 (Pin_4), U1.1 (ADDR), U1.3 (GND), U1.5 (AIN1)
- new net: C2.1, R1.2, U1.4 (AIN0)
- new net: D1.2 (A), R2.1
- new net GND: D1.1 (K), U2.3
- new net SCL: J1.2 (Pin_2), U1.10 (SCL), U2.1
- new net SDA: J1.3 (Pin_3), U1.9 (SDA), U2.2
- new net SIG: R1.1
