File: recovery/RecoveryModule/ChargeControl.kicad_sch (KiCad schematic)
At the start: 0 parts

Commit message: charge control schematics
Parts:
- added D1: MAIN_ACTIVE, symbol Device:LED
- added D2: DROGUE_ACTIVE, symbol Device:LED
- added D3, D4: D_TVS, Package_SON:WSON-6-1EP_2x2mm_P0.65mm_EP1x1.6mm, symbol Device:D_TVS
- added F1, F2: Polyfuse, symbol Device:Polyfuse
- added J1: DROGUE_EMATCH, symbol Connector_Generic:Conn_01x02
- added J2: MAIN_EMATCH, symbol Connector_Generic:Conn_01x02
- added Q1, Q2, Q3, Q4: NMOS, Package_DIP:DIP-24_W7.62mm, symbol Simulation_SPICE:NMOS
- added R10, R11, R12, R13, R14, R15, R4, R5, R6, R7, R8, R9: R, symbol Device:R
- added TP2: CMAIN, Relay_THT:Relay_DPDT_Schrack-RT2-FormC_RM5mm, symbol Connector:TestPoint
- added TP3: CDROGUE, Relay_THT:Relay_DPDT_Schrack-RT2-FormC_RM5mm, symbol Connector:TestPoint
Connections:
- new net: D3.1 (A1), J2.1 (Pin_1), Q1.1 (D), R7.1
- new net: Q1.2 (G), R4.1, R5.1
- new net: D4.1 (A1), J1.1 (Pin_1), Q3.1 (D), R11.2
- new net: F1.1, J1.2 (Pin_2)
- new net: Q2.2 (G), R7.2, R8.1
- new net: Q4.2 (G), R11.1, R13.1
- new net: D2.2 (A), R12.2
- new net: D1.2 (A), R6.1
- new net: Q3.2 (G), R10.1, R9.1
- new net: Q2.1 (D), R14.2
- new net: Q4.1 (D), R15.2
- new net: F2.1, J2.2 (Pin_2)
- new net +3.3V: R14.1, R15.1, TP2.1, TP3.1
- new net DROGUE_EN: R9.2
- new net GND: D1.1 (K), D2.1 (K), D3.2 (A2), D4.2 (A2), Q1.3 (S), Q2.3 (S), Q3.3 (S), Q4.3 (S), R10.2, R13.2, R5.2, R8.2
- new net MAIN_EN: R4.2
- new net VBATT: F1.2, F2.2, R12.1, R6.2
Other:
- title: STM32F1 Breakout Circuitry -> Charge Control
