File: recovery/RecoveryModule/STM32F1Breakout.kicad_sch (KiCad schematic)
At the start: 0 parts

Commit message: Added Breakout Circuitry
Parts:
- added C1: C, Package_SO:SOIC-8_3.9x4.9mm_P1.27mm, symbol Device:C
- added C2: C, symbol Device:C
- added R1, R2, R3: R, symbol Device:R
- added U1: STM32F103C8Tx, Package_QFP:LQFP-48_7x7mm_P0.5mm, symbol MCU_ST_STM32F1:STM32F103C8Tx
- added U2: CP2102N-Axx-xQFN28, Package_DFN_QFN:QFN-28-1EP_5x5mm_P0.5mm_EP3.35x3.35mm, symbol Interface_USB:CP2102N-Axx-xQFN28
Connections:
- new net: C2.1, R2.2, R3.1, U2.8 (VBUS)
- new net: R1.2, U2.9 (~{RST})
- new net +3.3V: C1.1, R1.1, U1.1 (VBAT), U1.24 (VDD), U1.36 (VDD), U1.48 (VDD), U2.6 (VDD), U2.7 (VREGIN)
- new net +3.3VA: U1.9 (VDDA)
- new net GND: C1.2, C2.2, R3.2, U1.23 (VSS), U1.35 (VSS), U1.47 (VSS), U1.8 (VSSA), U2.29 (GND), U2.3 (GND)
- new net STM_RESET: U1.7 (NRST)
- new net USB_D+: U2.4 (D+)
- new net USB_D-: U2.5 (D-)
- new net USB_RX: U2.26 (TXD)
- new net USB_TX: U1.30 (PA9), U2.25 (RXD)
- no-connect marks 0 -> 18

Commit message: charge control schematics
Other:
- moved on the sheet: C1, C2, R1, R2, R3, U1, U2
