File: recovery/RecoveryModule/SensorInterface.kicad_sch (KiCad schematic)
At the start: 0 parts

Commit message: sensor schematic
Parts:
- added C3, C4, C7, C8: 100n, symbol Device:C
- added C5, C6: 4u7, symbol Device:C
- added R4, R5: 4k7, symbol Device:R
- added R6, R7: 10k, symbol Device:R
- added U3: LPS27HHWTR, QFN_HHWTR_STM, symbol LPS27HHWTR:LPS27HHWTR
- added U4: LSM6DSV32XTR, LGA-14L_2p5X3p0X0p86_STM, symbol LSM6DSV32XTR:LSM6DSV32XTR
Connections:
- new net +3.3V: C3.1, C4.1, C5.1, C6.1, C7.1, C8.1, R4.1, R5.1, R6.1, R7.1, U3.1 (VDD_IO), U3.10 (VDD), U3.6 (CS), U4.12 (CS), U4.5 (VDD_IO), U4.8 (VDD)
- new net BARO_INT: U3.7 (INT_DRDY)
- new net BARO_SCL: R5.2, U3.2 (SCL/SPC)
- new net BARO_SDA: R4.2, U3.4 (SDA/SDI/SDO)
- new net GND: C3.2, C4.2, C5.2, C6.2, C7.2, C8.2, U3.11 (GND), U3.5 (SDO/SA0), U3.8 (GND), U3.9 (GND), U4.1 (SDO/SA0), U4.2 (SDX/AH1/QVAR1), U4.3 (SCX/AH2/QVAR2), U4.6 (GND), U4.7 (GND)
- new net IMU_INT: U4.4 (INT1)
- new net IMU_SCL: R6.2, U4.13 (SCL)
- new net IMU_SDA: R7.2, U4.14 (SDA)
- no-connect marks 0 -> 4

Commit message: charge control schematics
Parts:
- removed C3, C4, C7, C8: 100n, symbol Device:C
- removed C5, C6: 4u7, symbol Device:C
- removed R4, R5: 4k7, symbol Device:R
- removed R6, R7: 10k, symbol Device:R
- removed U3: LPS27HHWTR, QFN_HHWTR_STM, symbol LPS27HHWTR:LPS27HHWTR
- removed U4: LSM6DSV32XTR, LGA-14L_2p5X3p0X0p86_STM, symbol LSM6DSV32XTR:LSM6DSV32XTR
Connections:
- no-connect marks 4 -> 0
