File: recovery/RecoveryModule/SensorInterface.kicad_sch (KiCad schematic)
At the start: 12 parts, among them U3 LPS27HHWTR, U4 LSM6DSV32XTR

Commit message: add a little review note to be brought up at meeting
Other:
- note added: "review notes: - wires instead of labels for some passive connections, we will talk more about this on Sunday"
Changed lines of the file:
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@@
 		(comment 1 "Contributors: ")
+	)
+	(text "review notes:\n- wires instead of labels for some passive connections, \nwe will talk more about this on Sunday"
+		(exclude_from_sim no)
+		(at 216.408 28.194 0)
+		(effects
+			(font
+				(size 1.27 1.27)
+			)
+			(justify left)
+		)
 	)
 	(junction
